File: Q940.kicad_pcb (KiCad board)
At the start: 2 copper layers, 68.6 x 53.3 mm, 19 parts, among them J1 Power, J101 TO_HX711, J102 SHT-3x Temperature-1, J103 SHT-3x Temperature-2, J104 TO L298N MOTOR-DRIVER, J105 I2C LCD 16x2, J106 PWR_INPUT, J2 Digital/PWM, J3 Analog, J4 Digital/PWM

Commit message: とりあえずリリース
Parts:
- moved J104 0.16 mm to (153.3, 59.4)
Routing:
- net +5V: track 0.00 -> 155.1 mm
- net /SCL/A5: track 0.00 -> 61.6 mm
- net /SDA/A4: track 0.00 -> 56.3 mm
- net /*9: track 0.00 -> 10.9 mm
- net /8: track 0.00 -> 10.8 mm
- net /A1: track 0.00 -> 10.5 mm
- net /A0: track 0.00 -> 10.4 mm
- net /7: track 0.00 -> 10.2 mm
- net /*6: track 0.00 -> 10.2 mm
- net /*5: track 0.00 -> 10.2 mm
- added copper zone on B.Cu, net GND
Other:
- board text added: "2024 R000"
- board text added: "Q940 九州大学AMPSD"
- board text added: "SCL"
- board text added: "SDA"
