File: Q940.kicad_pcb (KiCad board)
At the start: 2 copper layers, 68.6 x 53.3 mm, 19 parts, among them J1 Power, J101 TO_HX711, J102 SHT-3x Temperature-1, J103 SHT-3x Temperature-2, J104 TO L298N MOTOR-DRIVER, J105 I2C LCD 16x2, J106 PWR_INPUT, J2 Digital/PWM, J3 Analog, J4 Digital/PWM

Commit message: append MPU6050 and Hardware interruption
Parts:
- added J107: MPU6050, Connector_JST:JST_XH_B4B-XH-A_1x04_P2.50mm_Vertical, F.Cu at (135.5, 72.0)
- added JP1: STOP1_SW, Jumper:SolderJumper-3_P1.3mm_Open_RoundedPad1.0x1.5mm_NumberLabels, F.Cu at (149.5, 55.6)
- added JP2: STOP2_SW, Jumper:SolderJumper-3_P1.3mm_Open_RoundedPad1.0x1.5mm_NumberLabels, F.Cu at (157.1, 55.6)
- J101: value TO_HX711 -> PWR_INPUT; footprint Connector_JST:JST_XH_B4B-XH-AM_1x04_P2.50mm_Vertical -> Connector_JST:JST_XH_B2B-XH-A_1x02_P2.50mm_Vertical
- J102: value SHT-3x Temperature-1 -> TO L298N MOTOR-DRIVER; footprint Connector_JST:JST_XH_B4B-XH-AM_1x04_P2.50mm_Vertical -> Connector_JST:JST_XH_B7B-XH-A_1x07_P2.50mm_Vertical
- J103: value SHT-3x Temperature-2 -> TO_HX711; footprint Connector_JST:JST_XH_B4B-XH-AM_1x04_P2.50mm_Vertical -> Connector_JST:JST_XH_B4B-XH-A_1x04_P2.50mm_Vertical
- J104: value TO L298N MOTOR-DRIVER -> LCD 16x2; footprint Connector_JST:JST_XH_B7B-XH-AM_1x07_P2.50mm_Vertical -> Connector_JST:JST_XH_B4B-XH-A_1x04_P2.50mm_Vertical
- J105: value I2C LCD 16x2 -> SHT-3x; footprint Connector_JST:JST_XH_B4B-XH-AM_1x04_P2.50mm_Vertical -> Connector_JST:JST_XH_B4B-XH-A_1x04_P2.50mm_Vertical
- J106: value PWR_INPUT -> SHT-3x; footprint Connector_JST:JST_XH_B2B-XH-AM_1x02_P2.50mm_Vertical -> Connector_JST:JST_XH_B4B-XH-A_1x04_P2.50mm_Vertical
- moved J101 41.1 mm to (103.8, 93.9), turned to 90 degrees
- moved J106 31.5 mm to (127.0, 72.0), turned to -90 degrees
- moved J103 23.7 mm to (150.5, 88.0), turned to 0 degrees
- moved J104 15.8 mm to (144.0, 72.1), turned to -90 degrees
- moved J102 11.2 mm to (153.2, 63.8), turned to 180 degrees
- moved C104 6.37 mm to (133.2, 63.8), turned to 90 degrees
- moved C103 3.39 mm to (158.0, 74.5)
- moved C105 0.40 mm to (138.1, 91.0), turned to 0 degrees
Connections:
- J101 pad 2: /A0 -> +5V
- J102 pad 2: +5V -> Net-(J102-Pin_2)
- J102 pad 3: /SDA/A4 -> Net-(J102-Pin_3)
- J102 pad 4: /SCL/A5 -> /7
- J103 pad 2: +5V -> /A0
- J103 pad 3: /SDA/A4 -> /A1
- J103 pad 4: /SCL/A5 -> +5V
- J104 pad 2: /*5 -> +5V
- J104 pad 3: /*6 -> /SDA/A4
- J104 pad 4: /7 -> /SCL/A5
Routing:
- net Net-(J102-Pin_2): track 0.00 -> 13.4 mm
- net +5V: track 155.1 -> 144.2 mm
- net /*3: track 0.00 -> 9.78 mm, vias 0 -> 1
- net Net-(J102-Pin_3): track 0.00 -> 8.72 mm
- net /2: track 0.00 -> 6.41 mm
- net /*9: track 10.9 -> 15.3 mm
- net /8: track 10.8 -> 15.3 mm
- net /7: track 10.2 -> 14.6 mm
- net /*6: track 10.2 -> 6.40 mm
- net /SDA/A4: track 56.3 -> 54.5 mm
- net /SCL/A5: track 61.6 -> 59.9 mm
Other:
- board text added: "2024 R100"
- board text added: "CLK"
- board text added: "DAT"
- board text added: "GND"
- board text added: "Vcc"
- board text removed: "2024 R000"
- board text removed: "ICSP"
